File: faceplate/midi_in_faceplate/midi_in_faceplate.kicad_pcb (KiCad board)
At the start: 2 copper layers, 98 x 30 mm, 0 parts

Commit message: Fill in metadata and put version number (v2.1.0b1) on the back silkscreen
Other:
- board text added: "v2.1.0b1"
Changed lines of the file:
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@@
   )
   (paper "A4")
+  (title_block
+    (title "MIDI IN Faceplate")
+    (date "2023-03-15")
+    (rev "2.1.0b1")
+    (company "Dave Dribin")
+  )
   (layers
     (0 "F.Cu" signal)
@@
   (gr_line locked (start 112.2832 92.5753) (end 112.7246 91.8388)
     (stroke (width 0.2) (type solid)) (layer "Edge.Cuts"))
+  (gr_text "v2.1.0b1" (at 187.5 111.5) (layer "B.SilkS")
+    (effects (font (size 1 1) (thickness 0.15)) (justify left bottom mirror))
+  )
   (gr_text "MIDI" (at 130.3325 85.95) (layer "F.SilkS")
     (effects (font (face "Arial Black") (size 2.5 2.5) (thickness 0.15)))
