File: faceplate/midi_out_faceplate/midi_out_faceplate.kicad_pcb (KiCad board)
At the start: 2 copper layers, 98 x 30 mm, 0 parts

Commit message: Fill in metadata and put version number (v2.1.0b1) on the back silkscreen
Other:
- board text added: "v2.1.0b1"
Changed lines of the file:
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@@
   )
   (paper "A4")
+  (title_block
+    (title "MIDI OUT Faceplate")
+    (date "2023-03-15")
+    (rev "2.1.0b1")
+    (company "Dave Dribin")
+  )
   (layers
     (0 "F.Cu" signal)
@@
   (gr_line locked (start 168.793 85.6181) (end 169.6423 85.4921)
     (stroke (width 0.2) (type solid)) (layer "Edge.Cuts"))
+  (gr_text "v2.1.0b1" (at 195 109) (layer "B.SilkS")
+    (effects (font (size 1 1) (thickness 0.15)) (justify left bottom mirror))
+  )
   (gr_text "Coupler" (at 170.5 106.7) (layer "F.SilkS")
     (effects (font (face "Arial Black") (size 2.5 2.5) (thickness 0.5) bold))
